Commit message: urdf file changed

File: wcr_description/urdf/wcr2.xacro (robot description, xacro)
@@ -22,5 +22,5 @@
             <origin rpy="0 ${-pi/2} ${pi}" xyz="0 0 0.01"/>
             <geometry>
-                <mesh filename="package://wcr_description/meshes/Housing_Electronic.stl" scale="0.001 0.001 0.001"/>
+                <mesh filename="package://wcr_description/meshes/robotChasiss.stl" scale="0.001 0.001 0.001"/>
             </geometry>
             <material name="gray"/>
@@ -35,14 +35,6 @@
     <link name="optitrack_link">
     </link>
-    <!-- IMU LINK - dobiven preko Optitrack-a...nije baš najbolje nanovo-->
+    <!-- IMU LINK -->
     <joint name="imu_joint" type="fixed">
-        <parent link="optitrack_link"/>
-        <child link="imu_link"/>
-        <origin xyz="0.031149 0.0140457 -0.0180142"/>
-    </joint>
-    <link name="imu_link">
-    </link>
-    <!-- IMU LINK -->
-    <!--<joint name="imu_joint" type="fixed">
         <parent link="base_link"/>
         <child link="imu_link"/>
@@ -50,5 +42,5 @@
     </joint>
     <link name="imu_link">
-    </link> -->
+    </link>
     <!-- T265 LINK -->
     <joint name="camera_joint" type="fixed">
@@ -58,14 +50,6 @@
     </joint>
     <link name="t265_link">
-        <visual>
-			<origin rpy="${pi/2} 0 0" xyz="-0.01225 0.0449 -0.0125 "/>
-			<geometry>
-			    <mesh filename="package://wcr_description/meshes/rs_t265.stl" scale="0.001 0.001 0.001"/>
-			</geometry>
-			<material name="yellow"/>
-		</visual>
     </link>
     <!-- MARVELMIND LINK -->
-    <!-- <origin xyz="-0.1307 0.002 0.1267"/> -->
     <joint name="marvelmind_joint" type="fixed">
         <parent link="base_link"/>
@@ -74,27 +58,5 @@
     </joint>
     <link name="marvelmind_link">
-        <visual>
-            <origin rpy="0 0 ${-pi/2}" xyz="-0.027 0 0"/>
-            <geometry>
-                <mesh filename="package://wcr_description/meshes/mm_beacon.stl" scale="0.001 0.001 0.001"/>
-            </geometry>
-            <material name="yellow"/>
-        </visual>
     </link>
-    <!-- CHASSIS LINK -->
-    <!--<joint name="chassis_joint" type="fixed">
-        <parent link="base_link"/>
-        <child link="chassis"/>
-        <origin xyz="-0 0 0.01"/>
-    </joint>
-    <link name="chassis">
-        <visual>
-            <origin rpy="0 ${-pi/2} ${pi}" xyz="0 0 0"/>
-            <geometry>
-                <mesh filename="package://wcr_description/meshes/Housing_Electronic.stl" scale="0.001 0.001 0.001"/>
-            </geometry>
-            <material name="gray"/>
-        </visual>
-    </link>-->
     <!-- FRONT LEFT SYSTEM -->
     <joint name="FL_steering" type="revolute">

Commit message: novi stl

File: wcr_description/urdf/wcr2.xacro (robot description, xacro)
@@ -17,8 +17,8 @@
         <color rgba="1 1 0 1"/>
     </material>
-    <!-- BASE LINK proba s dualboota-->
+    <!-- BASE LINK -->
     <link name="base_link">
         <visual>
-            <origin rpy="0 ${-pi/2} ${pi}" xyz="0 0 0.01"/>
+            <origin rpy="0 0 0" xyz="0 0 0.01"/>
             <geometry>
                 <mesh filename="package://wcr_description/meshes/robotChasiss.stl" scale="0.001 0.001 0.001"/>

Commit message: changed urdf file with new dimensions

File: wcr_description/urdf/wcr2.xacro (robot description, xacro)
@@ -3,5 +3,5 @@
     <xacro:property name="length" value="0.225" />
 	<xacro:property name="width" value="0.225" />
-	<xacro:property name="steering_height" value="0.06029" />
+	<xacro:property name="steering_height" value="0.05029" />
 	<xacro:property name="wheel_height" value="-0.035250" />
     <material name="gray">
@@ -20,5 +20,5 @@
     <link name="base_link">
         <visual>
-            <origin rpy="0 0 0" xyz="0 0 0.01"/>
+            <origin rpy="0 0 0" xyz="0 0 0.0103600017"/>
             <geometry>
                 <mesh filename="package://wcr_description/meshes/robotChasiss.stl" scale="0.001 0.001 0.001"/>
