Commit message: urdf change

File: wcr_description/urdf/wcr.xacro (robot description, xacro)
@@ -3,5 +3,5 @@
     <xacro:property name="length" value="0.225" />
 	<xacro:property name="width" value="0.225" />
-	<xacro:property name="steering_height" value="0.05029" />
+	<xacro:property name="steering_height" value="0.0606500017" /> <!--STEERING HEIGHT + OFFSET FROM BASE LINK TO CHASSIS-->
 	<xacro:property name="wheel_height" value="-0.035250" />
     <material name="gray">
@@ -19,43 +19,51 @@
     <!-- BASE LINK -->
     <link name="base_link">
-        <visual>
-            <origin rpy="0 0 0" xyz="0 0 0.0103600017"/>
+    </link>
+    <!-- OPTITRACK LINK -->
+    <joint name="optitrack_joint" type="fixed">
+        <parent link="base_link"/>
+        <child link="optitrack_link"/>
+        <origin xyz="0 0 0.120"/> <!--140 mjerenjem, 120 iz optitrack-a-->
+    </joint>
+    <link name="optitrack_link">
+    </link>
+    <!-- IMU LINK -->
+    <joint name="imu_joint" type="fixed">
+        <parent link="base_link"/>
+        <child link="imu_link"/>
+        <origin xyz="0.06579 0 0.08934"/>
+    </joint>
+    <link name="imu_link">
+    </link>
+    <!-- T265 LINK -->
+    <joint name="camera_joint" type="fixed">
+        <parent link="base_link"/>
+        <child link="t265_link"/>
+        <origin xyz="0.16 0 0.075"/>
+    </joint>
+    <link name="t265_link">
+    </link>
+    <!-- MARVELMIND LINK -->
+    <joint name="marvelmind_joint" type="fixed">
+        <parent link="base_link"/>
+        <child link="marvelmind_link"/>
+        <origin xyz="-0.1223 0.000 0.1205"/>
+    </joint>
+    <link name="marvelmind_link">
+    </link>
+    <!-- CHASSIS LINK-->
+    <joint name="chassis_joint" type="fixed">
+        <parent link="base_link"/>
+        <child link="chassis_link"/>
+        <origin xyz="0 0 0.0103600017"/>
+    </joint>
+    <link name="chassis_link">
+        <visual>
+            <origin rpy="0 0 0" xyz="0 0 0"/>
             <geometry>
-                <mesh filename="package://wcr_description/meshes/robotChasiss.stl" scale="0.001 0.001 0.001"/>
+                <mesh filename="package://wcr_description/meshes/robotChassis.stl" scale="0.001 0.001 0.001"/>
             </geometry>
             <material name="gray"/>
         </visual>
-    </link>
-    <!-- OPTITRACK LINK -->
-    <joint name="optitrack_joint" type="fixed">
-        <parent link="base_link"/>
-        <child link="optitrack_link"/>
-        <origin xyz="0 0 0.120"/> <!--140 mjerenjem, 120 iz optitrack-a-->
-    </joint>
-    <link name="optitrack_link">
-    </link>
-    <!-- IMU LINK -->
-    <joint name="imu_joint" type="fixed">
-        <parent link="base_link"/>
-        <child link="imu_link"/>
-        <origin xyz="0.06579 0 0.08934"/>
-    </joint>
-    <link name="imu_link">
-    </link>
-    <!-- T265 LINK -->
-    <joint name="camera_joint" type="fixed">
-        <parent link="base_link"/>
-        <child link="t265_link"/>
-        <origin xyz="0.16 0 0.075"/>
-    </joint>
-    <link name="t265_link">
-    </link>
-    <!-- MARVELMIND LINK -->
-    <joint name="marvelmind_joint" type="fixed">
-        <parent link="base_link"/>
-        <child link="marvelmind_link"/>
-        <origin xyz="-0.1223 0.000 0.1205"/>
-    </joint>
-    <link name="marvelmind_link">
     </link>
     <!-- FRONT LEFT SYSTEM -->

Commit message: urdf change

File: wcr_description/urdf/wcr.xacro (robot description, xacro)
@@ -3,5 +3,5 @@
     <xacro:property name="length" value="0.225" />
 	<xacro:property name="width" value="0.225" />
-	<xacro:property name="steering_height" value="0.0606500017" /> <!--STEERING HEIGHT + OFFSET FROM BASE LINK TO CHASSIS-->
+	<xacro:property name="steering_height" value="0.05029" />
 	<xacro:property name="wheel_height" value="-0.035250" />
     <material name="gray">
@@ -30,5 +30,5 @@
     <!-- IMU LINK -->
     <joint name="imu_joint" type="fixed">
-        <parent link="base_link"/>
+        <parent link="chassis_link"/>
         <child link="imu_link"/>
         <origin xyz="0.06579 0 0.08934"/>
@@ -38,5 +38,5 @@
     <!-- T265 LINK -->
     <joint name="camera_joint" type="fixed">
-        <parent link="base_link"/>
+        <parent link="chassis_link"/>
         <child link="t265_link"/>
         <origin xyz="0.16 0 0.075"/>
@@ -46,5 +46,5 @@
     <!-- MARVELMIND LINK -->
     <joint name="marvelmind_joint" type="fixed">
-        <parent link="base_link"/>
+        <parent link="chassis_link"/>
         <child link="marvelmind_link"/>
         <origin xyz="-0.1223 0.000 0.1205"/>
@@ -70,5 +70,5 @@
     <joint name="FL_steering" type="revolute">
         <limit effort="100.0" lower="${-pi/2}" upper="${pi/2}" velocity="5.23598775"/>
-        <parent link="base_link"/>
+        <parent link="chassis_link"/>
         <child link="FL_steering_link"/>
         <origin xyz="${length/2} ${width/2} ${steering_height}"/>
@@ -103,5 +103,5 @@
     <joint name="BL_steering" type="revolute">
         <limit effort="100.0" lower="${-pi/2}" upper="${pi/2}" velocity="5.23598775"/>
-        <parent link="base_link"/>
+        <parent link="chassis_link"/>
         <child link="BL_steering_link"/>
         <origin xyz="-${length/2} ${width/2} ${steering_height}"/>
@@ -136,5 +136,5 @@
     <joint name="BR_steering" type="revolute">
         <limit effort="100.0" lower="${-pi/2}" upper="${pi/2}" velocity="5.23598775"/>
-        <parent link="base_link"/>
+        <parent link="chassis_link"/>
         <child link="BR_steering_link"/>
         <origin xyz="-${length/2} -${width/2} ${steering_height}"/>
@@ -169,5 +169,5 @@
     <joint name="FR_steering" type="revolute">
         <limit effort="100.0" lower="${-pi/2}" upper="${pi/2}" velocity="5.23598775"/>
-        <parent link="base_link"/>
+        <parent link="chassis_link"/>
         <child link="FR_steering_link"/>
         <origin xyz="${length/2} -${width/2} ${steering_height}"/>

Commit message: last update

File: wcr_description/urdf/wcr.xacro (robot description, xacro)
@@ -32,5 +32,5 @@
         <parent link="chassis_link"/>
         <child link="imu_link"/>
-        <origin xyz="0.06579 0 0.08934"/>
+        <origin xyz="0.06551 0 0.098"/>
     </joint>
     <link name="imu_link">

Commit message: t265_link new dimensions

File: wcr_description/urdf/wcr.xacro (robot description, xacro)
@@ -40,5 +40,5 @@
         <parent link="chassis_link"/>
         <child link="t265_link"/>
-        <origin xyz="0.16 0 0.075"/>
+        <origin xyz="0.14885 0.00922 0.05459"/>
     </joint>
     <link name="t265_link">

Commit message: added some rs stuff

File: wcr_description/urdf/wcr.xacro (robot description, xacro)
@@ -43,4 +43,12 @@
     </joint>
     <link name="t265_link">
+    </link>
+    <!-- T265 ODOM -->
+    <joint name="camera_odom_joint" type="fixed">
+        <parent link="chassis_link"/>
+        <child link="t265_odom_frame"/>
+        <origin xyz="0.14885 0.00922 0.05459"/>
+    </joint>
+    <link name="t265_odom_frame">
     </link>
     <!-- MARVELMIND LINK -->

Commit message: added display_dummy and change chasiss name

File: wcr_description/urdf/wcr.xacro (robot description, xacro)
@@ -40,5 +40,5 @@
         <parent link="chassis_link"/>
         <child link="t265_link"/>
-        <origin xyz="0.14885 0.00922 0.05459"/>
+        <origin xyz="0.14885 0.00922 0.06659"/>
     </joint>
     <link name="t265_link">
@@ -48,5 +48,5 @@
         <parent link="chassis_link"/>
         <child link="t265_odom_frame"/>
-        <origin xyz="0.14885 0.00922 0.05459"/>
+        <origin xyz="0.14885 0.00922 0.06659"/>
     </joint>
     <link name="t265_odom_frame">
@@ -70,5 +70,5 @@
             <origin rpy="0 0 0" xyz="0 0 0"/>
             <geometry>
-                <mesh filename="package://wcr_description/meshes/robotChassis.stl" scale="0.001 0.001 0.001"/>
+                <mesh filename="file://$(find wcr_description)/meshes/robotChasissNew.stl" scale="0.001 0.001 0.001"/>
             </geometry>
             <material name="gray"/>
